File: P3_MP3player.kicad_sch (KiCad schematic)
At the start: 34 parts, among them J101 USB_C_Receptacle_USB2.0, SW201 PowerON, SW205 SW_Push, U1 USBLC6-2SC6, U201 PCM5102A, U202 Microchip_BM83, U203 ST7735S, U204 STM32G431KBTx

Commit message: 回路図ひとまず完成
Parts:
- removed C201, C204: 2.2n, Capacitor_SMD:C_0603_1608Metric, symbol Device:C_Small
- removed C202, C203: 1u, Capacitor_THT:C_Rect_L7.2mm_W6.0mm_P5.00mm, symbol Device:C_Small
- removed C205, C212: 2.2u, Capacitor_SMD:C_0603_1608Metric, symbol Device:C_Small
- removed C206, C208, C210, C213: 0.1u, Capacitor_SMD:C_0603_1608Metric, symbol Device:C_Small
- removed C207, C209, C211, C214: 10u, Capacitor_SMD:CP_Elec_3x5.3, symbol Device:C_Polarized_Small
- removed C215: 0.1u, Capacitor_SMD:C_0603_1608Metric, symbol Device:C
- removed C216, C219: 0.1u, Capacitor_SMD:C_0402_1005Metric, symbol Device:C
- removed C217: 0.01u, Capacitor_SMD:C_0402_1005Metric, symbol Device:C
- removed C218: 4.7u, Capacitor_SMD:C_0402_1005Metric, symbol Device:C
- removed FB101: 60, Inductor_SMD:L_0603_1608Metric, symbol Device:FerriteBead_Small
- removed R201, R204: 100k, Resistor_SMD:R_0603_1608Metric, symbol Device:R_Small
- removed R202, R203: 470, Resistor_SMD:R_0603_1608Metric, symbol Device:R_Small
- removed R205, R206: 10k, Resistor_SMD:R_0603_1608Metric, symbol Device:R_Small
- removed SW201: PowerON, Connector_JST:JST_XH_B2B-XH-A_1x02_P2.50mm_Vertical, symbol Switch:SW_SPST
- removed SW205: SW_Push, samacsys:TVAF06A020BR, symbol Switch:SW_Push
- removed U201: PCM5102A, Package_SO:TSSOP-20_4.4x6.5mm_P0.65mm, symbol Audio:PCM5102A
- removed U203: ST7735S, Connector_JST:JST_XH_B8B-XH-A_1x08_P2.50mm_Vertical, symbol MysymbolLibrary:ST7735S
- removed U204: STM32G431KBTx, Package_QFP:LQFP-32_7x7mm_P0.8mm, symbol MCU_ST_STM32G4:STM32G431KBTx
- added C1, C4, C5: 0.1u, Package_SON:WSON-8-1EP_6x5mm_P1.27mm_EP3.4x4mm, symbol Device:C_Small
- added C2: 1u, Package_SON:WSON-8-1EP_6x5mm_P1.27mm_EP3.4x4mm, symbol Device:C_Small
- added C3: 4.7u, Package_SON:WSON-8-1EP_6x5mm_P1.27mm_EP3.4x4mm, symbol Device:C_Small
- added D1, D2: LED, symbol Device:LED_Small
- added F1, F2: Fuse, Package_QFP:LQFP-100_14x14mm_P0.5mm, symbol Device:Fuse_Polarized_Small
- added J1: BATT, symbol Connector_Generic:Conn_01x02
- added J2: FH12-8S-0.5SH(55), Package_DFN_QFN:Nordic_AQFN-94-1EP_7x7mm_P0.4mm, symbol Connector_Generic:Conn_01x08
- added J4: Write, Package_DFN_QFN:Nordic_AQFN-94-1EP_7x7mm_P0.4mm, symbol Connector_Generic:Conn_01x03
- added J5: AudioJack3, MyLibrary:MJ352W, symbol Connector_Audio:AudioJack3
- added Q1: PNP, Package_DIP:DIP-24_W7.62mm, symbol Simulation_SPICE:PNP
- added Q2: NPN, symbol Simulation_SPICE:NPN
- added R1, R3: 100k, Resistor_SMD:R_0603_1608Metric, symbol Device:R_Small
- added R10, R4: 1k, Resistor_SMD:R_0603_1608Metric, symbol Device:R_Small
- added R2, R8: 10k, Resistor_SMD:R_0603_1608Metric, symbol Device:R_Small
- added R5: 10, Resistor_SMD:R_0603_1608Metric, symbol Device:R_Small
- added R6, R7: 5.1k, Resistor_SMD:R_0603_1608Metric, symbol Device:R_Small
- added R9: 20k, Resistor_SMD:R_0603_1608Metric, symbol Device:R_Small
- added SW1, SW2, SW3, SW4, SW5, SW6: PowerON, Connector_JST:JST_XH_B2B-XH-A_1x02_P2.50mm_Vertical, symbol Switch:SW_SPST
- added SW7: RST_N, Connector_JST:JST_XH_B2B-XH-A_1x02_P2.50mm_Vertical, symbol Switch:SW_SPST
- added SW8: NRST, Connector_JST:JST_XH_B2B-XH-A_1x02_P2.50mm_Vertical, symbol Switch:SW_SPST
- added U2: RT9080-33GJ5, Package_TO_SOT_SMD:SOT-23-5, symbol NITTC_Robocon_Library:RT9080-33GJ5
- added U4: CH32V003F4P6, symbol MysymbolLibrary:CH32V003F4P6
- renumbered J101 to J3, U202 to U3
Connections:
- net GNDD is gone; now on net GND: J3.A1 (GND), J3.A12 (GND), J3.B1 (GND), J3.B12 (GND), U1.2 (GND), U3.16 (GND), U3.50 (GND), U3.56 (GND), U3.57 (GND)
- net +3.3V: now also C1.1, C3.1, C5.2, J2.3 (Pin_3), J2.7 (Pin_7), J4.1 (Pin_1), Q1.3 (E), R2.1, R9.1, U2.5 (OUT), U4.9 (VDD)
- net +5V: now also U1.5 (VBUS), F2.2
- net AOHPL: now also J5.T
- net AOHPM: now also J5.S
- net AOHPR: now also J5.R
- net D+: now also U1.4 (I/O2), U3.37 (DP); no longer U1.6 (I/O1), U3.36 (DM)
- net D-: now also U1.6 (I/O1), U3.36 (DM); no longer U1.4 (I/O2), U3.37 (DP)
- net GND: now also C1.2, C2.2, C3.2, C4.2, C5.1, J1.2 (Pin_2), J2.2 (Pin_2), J2.8 (Pin_8), J4.2 (Pin_2), Q2.3 (E), R3.2, R6.2, R7.2, R8.2, SW2.1 (A), SW3.1 (A), SW4.1 (A), SW5.1 (A), SW6.1 (A), SW7.1 (A), SW8.1 (A), U2.2 (GND), U4.6 (PA2/OSCO/A0/T1CH2N/OPP0/AETR2_), U4.7 (VSS)
- net MOSI: now also J2.5 (Pin_5), U4.16 (PC6/MOSI/T1CH1CH3N_/UCTS_/SDA_)
- net SCK: now also J2.6 (Pin_6), U4.15 (PC5/SCK/T1ETR/T2CH1ETR_/SCL_/UCK_/T1CH3_)
- net ~{RST}: now also SW7.2 (B)
- net PWR(MFB): now reaches U3.26 (PWR(MFB))
- net PWR(MFB): now also R10.1, R8.1, SW1.1 (A)
- net at J3.A5 (CC1): now also R7.1
- net at J3.B5 (CC2): now also R6.1
- net +BATT: now reaches U3.23 (BAT_IN)
- net +BATT: now also C2.1, F1.2, R1.1, U2.1 (IN), U2.3 (EN)
- net SYS_PWR: now reaches U3.24 (SYS_PWR)
- net SYS_PWR: now also D1.2 (A), D2.2 (A), SW1.2 (B)
- net BCK: no longer names the net of U3.3 (SCLK1)
- net DIN: no longer names the net of U3.4 (DT1)
- net LED1: no longer names the net of U3.32 (LED1)
- net LED1: now also D1.1 (K)
- net LED2: no longer names the net of U3.34 (LED2)
- net LED2: now also D2.1 (K)
- net LRCK: no longer names the net of U3.2 (RFS1)
- net UART_RX_STM renamed UART_RX_CH32
- net UART_RX_CH32: now also U4.2 (PD5/A5/UTX/T2CH4_/URX_)
- net UART_TX_STM renamed UART_TX_CH32
- net UART_TX_CH32: now also U4.3 (PD6/A6/URX/T2CH3_/UTX_)
- net VBUS: no longer names the net of J3.A4 (VBUS), J3.A9 (VBUS), J3.B4 (VBUS), J3.B9 (VBUS)
- net VBUS: now also F2.1; no longer U1.5 (VBUS)
- net external codec reset: no longer names the net of U3.49 (P0_0/UART_TX_IND)
- net foward renamed FWD
- net FWD: now also SW2.2 (B)
- net play/pause renamed PLAY/PAUSE
- net PLAY/PAUSE: now also SW4.2 (B)
- net reverse renamed REV
- net REV: now also SW3.2 (B)
- net volume_down renamed VOL_DN
- net VOL_DN: now also SW6.2 (B)
- net volume_up renamed VOL_UP
- net VOL_UP: now also SW5.2 (B)
- new net: C4.1, SW8.2 (B), U4.4 (PD7/NRST/T2CH4/OPP1/UCK_)
- new net: Q1.2 (B), R2.2, R4.2
- new net: Q1.1 (C), R5.1
- new net: Q2.2 (B), R10.2
- new net: F1.1, J1.1 (Pin_1)
- new net BATT_V: R1.2, R3.1, U4.5 (PA1/OSCI/A1/T1CH2/OPN0)
- new net BLK: R4.1, U4.13 (PC3/T1CH3/T1CH1N_/UCTS_)
- new net LEDA: J2.1 (Pin_1), R5.2
- new net RS: J2.4 (Pin_4), U4.14 (PC4/A2/T1CH4/MCO/T1CH1CH2N_)
- new net SWIO: J4.3 (Pin_3), U4.18 (PD1/SWIO/AETR2/T1CH3N/SCL_/URX_)
- new net ~{PWR_STATE}: Q2.1 (C), R9.2, U4.10 (PC0/T2CH3/UTX_/NSS_/T1CH3_)
- no-connect marks 37 -> 31
Other:
- note added: "BATT"
- note added: "BM83 WRIET & BATT CHARGE"
- note added: "Current:600mA DO:310mV"
- note added: "Digikey"
- note added: "EARPHONES"
- note added: "I/F"
- note added: "LCD"
- note added: "LCD 62.5*17.9 これから剥がす"
- note added: "LCD表示内容 ・BT接続状況 ・電池残量 ・曲名 ・アーティスト名 ・音量 ．再生/一時停止 ．楽曲時間"
- note added: "LDO"
- note added: "LEVEL CONV"
- note added: "Lipo 50*20*10 1000mAh"
- note added: "Lipo 約102*25*4 でかいな"
- note added: "MCU WRITE"
- note added: "USB2.0規格準拠：5V500mA →BM83の充電機能は350mAらしい"
- note added: "回路図の都合上同一ラベルとしているが， 書き込み時は独自の外部電源である点に留意"
- note added: "物理IFは ・電源 ・前/次の曲 ・再生 ・一時停止"
- note added: "要容量計算"
- note removed: "1cell 3.7V→Boost DC/DC→6V程度？ 片電源or両電源？→楽に省面積でやるなら片電源 EQいる? UACつける？ いずれにしてもUSBはBM83書き込みのためにいる キャラクタディスプレイ何出す？ 文字しか出せない，文字以外出したければLCD UACいらないならRISC-Vでいい イヤホン駆動だけならPCM5102Aもいらない PCM5102Aつけるなら電流増幅段もいる"
- note removed: "BM83のみならここから出力"
- note removed: "BM83のみなら不要"
- note removed: "PCM5102A"
- note removed: "書き込み"
- note removed: "物理IFは ・電源 ・前/次の曲 ・再生 ・一時停止 →ボタン機能重複の兼ね合いから，BM83オンリーでいいかも"
- moved on the sheet: J3, U1
